File: kicad/shield_gas_sensor/shield_gas_sensor.kicad_sch (KiCad schematic)
At the start: 16 parts, among them P1 Power, P2 Analog, P3 Digital, P4 Digital, P5 CONN_01X01, P6 CONN_01X01, P7 CONN_01X01, P8 CONN_01X01

Commit message: Kicad improvements
Parts:
- added C2, C3: 100n, symbol Device:C
- added C4: 1u, symbol Device:C
- added U2: RN2463, symbol lora_module:RN2463
- 10k: renamed from R?; value R -> R5
- C1: renamed from C?; value C -> 100n
- R1, R3: renamed from R?; value R -> 100k
- R2, R6: renamed from R?; value R -> 1k
- gave numbers to parts that had none: 2
Connections:
- net +3V3: now also U2.6 (3V3)
- net +5V: now also S1.2 (gas1_a), S1.3 (heater_1), U1.7 (V+), C3.1
- net GND: now also S1.6 (temp_2), S1.8 (heater_2), C2.2, C3.2, U2.8 (GND)
- net at R2.2, U1.2 (-IN): now also R3.2, C4.1
- net at R6.2, U1.6 (OUT): now also R3.1, C4.2
- net at R6.1: now also C2.1
- net Gas_sensor: now reaches S1.4 (gas1_b)
- net Gas_sensor: now also 10k.2
- new net RST_LoRa: U2.5 (RST)
- new net Rx_LoRa: U2.2 (RX)
- new net Tx_LoRa: U2.1 (TX)
- no-connect marks 5 -> 14
Other:
- moved on the sheet: 10k, C1, R1, R2, R3, R6, S1, U1
