File: kicad_francois/shield_gas_sensor/shield_gas_sensor.kicad_pcb (KiCad board)
At the start: 2 copper layers, 69.6 x 55 mm, 26 parts, among them J1 Screw_Terminal_01x02, J2 Grove gas MQx, J3 Lora RN2483 Module, J4 Jumper sensor choice, J5 Jumper sensor choice, P1 Power, P2 Analog, P3 Digital, P4 Digital, P6 CONN_01X01, P7 CONN_01X01, P8 CONN_01X01, U1 LTC_1050

Commit message: mise a jour Readme et Kicad
Parts:
- moved JP2 5.09 mm to (165.1, 118.5)
- moved JP3 4.58 mm to (162.3, 118.5)
Routing:
- net GND: track 210.4 -> 221.0 mm
- net /A0: track 16.9 -> 26.3 mm
- net /A1: track 73.0 -> 79.9 mm
- net +3V3: track 143.8 -> 147.5 mm
Other:
- board text added: "Bottom Implantation"
- board text added: "BottomLayer"
- board text added: "BottomOverlay"
- board text added: "Dimensions"
- board text added: "GROVE"
- board text added: "NANO"
- board text added: "SEED"
- board text added: "SENSOR"
- board text added: "Top Implantation"
- board text added: "TopLayer"
- board text added: "TopOverlay"
